Commit message: 実機とシミュレーション使い分けれるように変更

File: config/so101_new_calib.ros2_control.xacro (robot description, xacro)
@@ -1,10 +1,15 @@
 <?xml version="1.0"?>
 <robot xmlns:xacro="http://www.ros.org/wiki/xacro">
-    <xacro:macro name="so101_new_calib_ros2_control" params="name initial_positions_file">
+    <xacro:macro name="so101_new_calib_ros2_control" params="name initial_positions_file use_sim:=true">
         <xacro:property name="initial_positions" value="${load_yaml(initial_positions_file)['initial_positions']}"/>
         <ros2_control name="${name}" type="system">
             <hardware>
-                <plugin>feetech_ros2_driver/FeetechHardwareInterface</plugin>
-                <param name="usb_port">/dev/serial/by-id/usb-1a86_USB_Single_Serial_5AF7133194-if00</param>
+                <xacro:if value="${use_sim}">
+                    <plugin>mock_components/GenericSystem</plugin>
+                </xacro:if>
+                <xacro:unless value="${use_sim}">
+                    <plugin>feetech_ros2_driver/FeetechHardwareInterface</plugin>
+                    <param name="usb_port">/dev/serial/by-id/usb-1a86_USB_Single_Serial_5AF7133194-if00</param>
+                </xacro:unless>
             </hardware>
             <joint name="shoulder_pan">

File: config/so101_new_calib.urdf.xacro (robot description, xacro)
@@ -2,8 +2,16 @@
 <robot xmlns:xacro="http://www.ros.org/wiki/xacro" name="so101_new_calib">
     <xacro:arg name="initial_positions_file" default="initial_positions.yaml" />
+    <xacro:arg name="use_sim" default="true" />
     <!-- Import so101_new_calib urdf file -->
     <xacro:include filename="$(find vla_manipulator)/models/robot.urdf" />
     <!-- Import control_xacro -->
     <xacro:include filename="so101_new_calib.ros2_control.xacro" />
-    <xacro:so101_new_calib_ros2_control name="FakeSystem" initial_positions_file="$(arg initial_positions_file)"/>
+    <xacro:so101_new_calib_ros2_control name="FakeSystem" initial_positions_file="$(arg initial_positions_file)" use_sim="$(arg use_sim)"/>
+    <xacro:if value="$(arg use_sim)">
+        <gazebo>
+            <plugin filename="ign_ros2_control-system" name="ign_ros2_control::IgnitionROS2ControlPlugin">
+                <parameters>$(find vla_manipulator_sim)/config/ros2_controllers.yaml</parameters>
+            </plugin>
+        </gazebo>
+    </xacro:if>
 </robot>

Commit message: 変更

File: config/so101_new_calib.ros2_control.xacro (robot description, xacro)
@@ -1,15 +1,18 @@
 <?xml version="1.0"?>
 <robot xmlns:xacro="http://www.ros.org/wiki/xacro">
-    <xacro:macro name="so101_new_calib_ros2_control" params="name initial_positions_file use_sim:=true">
-        <xacro:property name="initial_positions" value="${load_yaml(initial_positions_file)['initial_positions']}"/>
+    <xacro:macro name="so101_new_calib_ros2_control" params="name initial_positions_file hardware_type:=mock">
+        <xacro:property name="initial_positions" value="${xacro.load_yaml(initial_positions_file)['initial_positions']}"/>
         <ros2_control name="${name}" type="system">
             <hardware>
-                <xacro:if value="${use_sim}">
+                <xacro:if value="${hardware_type == 'mock'}">
                     <plugin>mock_components/GenericSystem</plugin>
                 </xacro:if>
-                <xacro:unless value="${use_sim}">
+                <xacro:if value="${hardware_type == 'gazebo'}">
+                    <plugin>ign_ros2_control/IgnitionSystem</plugin>
+                </xacro:if>
+                <xacro:if value="${hardware_type == 'real'}">
                     <plugin>feetech_ros2_driver/FeetechHardwareInterface</plugin>
                     <param name="usb_port">/dev/serial/by-id/usb-1a86_USB_Single_Serial_5AF7133194-if00</param>
-                </xacro:unless>
+                </xacro:if>
             </hardware>
             <joint name="shoulder_pan">

File: config/so101_new_calib.urdf.xacro (robot description, xacro)
@@ -2,11 +2,11 @@
 <robot xmlns:xacro="http://www.ros.org/wiki/xacro" name="so101_new_calib">
     <xacro:arg name="initial_positions_file" default="initial_positions.yaml" />
-    <xacro:arg name="use_sim" default="true" />
+    <xacro:arg name="hardware_type" default="mock" />
     <!-- Import so101_new_calib urdf file -->
     <xacro:include filename="$(find vla_manipulator)/models/robot.urdf" />
     <!-- Import control_xacro -->
     <xacro:include filename="so101_new_calib.ros2_control.xacro" />
-    <xacro:so101_new_calib_ros2_control name="FakeSystem" initial_positions_file="$(arg initial_positions_file)" use_sim="$(arg use_sim)"/>
-    <xacro:if value="$(arg use_sim)">
+    <xacro:so101_new_calib_ros2_control name="FakeSystem" initial_positions_file="$(arg initial_positions_file)" hardware_type="$(arg hardware_type)"/>
+    <xacro:if value="${'gazebo' == '$(arg hardware_type)'}">
         <gazebo>
             <plugin filename="ign_ros2_control-system" name="ign_ros2_control::IgnitionROS2ControlPlugin">
